File: pcb/tvbgone3.brd (EAGLE design)
At the start: 36.8 x 57.1 mm, 32 parts, among them Q1 MMBT5088, Q2 MMBT5088, Q3 MMBT5088, Q4 MMBT5088, Q5 MMBT4403, Q6 MOSFET-NCHANNELBSS123LT1G, Q7 MOSFET-NCHANNELBSS123LT1G, U1 ATTINY85V-10SU, U3 MCP73831

Commit message: finalized version 1 of smd board and documented the fuses. Tested. It Works\!
Parts:
- C4: value 0.22uF -> 4.7uF
- C5: value 0.22uF -> 0.1uF
- R1: value 2.0M -> 1K
- R2: value 2.0M -> 10k(opt)
- R3: value (none) -> 1k
- R4: value (none) -> 2K
- R5: value 2.0M -> 1k
- R6: value (none) -> 1K
